File: quark-u5-som/microcontroller.kicad_sch (KiCad schematic)
At the start: 0 parts

Commit message: Add .ioc
Parts:
- added C1, C2, C3: 4.7uF, symbol Device:C
- added C4, C5, C6, C7, C8: 100nF, symbol Device:C
- added L1: L, symbol Device:L
- added U1: STM32U535VCTxQ, Package_QFP:LQFP-100_14x14mm_P0.5mm, symbol MCU_ST_STM32U5:STM32U535VCTxQ
Connections:
- new net: U1.10 (VSS), U1.26 (VSS), U1.50 (VSS), U1.74 (VSS), U1.99 (VSS)
- new net +3.3V: C2.1, C3.1, C4.1, C5.1, C6.1, C7.1, C8.1, L1.2
- new net +3.3VA: C1.1, L1.1
- new net GNDD: C1.2, C2.2, C3.2, C4.2, C5.2, C6.2, C7.2, C8.2
